File: pcb/musicbox/eagle/musicbox.brd (EAGLE design)
At the start: 67.3 x 68.5 mm, 17 parts, among them J1 1727010, J2 22-27-2031-03, J3 22-27-2021-02, J4 22-27-2021-02, J5 22-27-2051-05, T1 2N2222

Commit message: added gerber files
Parts:
- added SJ1: No Addon, jumper:SJW
Connections:
- net A10: now also SJ1.2
- net N$15: now also SJ1.1
Routing:
- net N$15: track 53.4 -> 59.8 mm
- net A10: track 70.0 -> 76.4 mm
Other:
- board text added: "J3-pins must be shorted (or SJ1 closed) if connector is not used"
- board text removed: "J3-pins must be shorted if connector is unused"
Changed lines of the file:
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@@
 <text x="6.35" y="31.75" size="1.016" layer="25" ratio="12" align="center">MIDI-PLAYER
 ADD-ON</text>
-<text x="64.77" y="56.515" size="1.016" layer="25" ratio="12" distance="39" rot="R90" align="center-left">NOTE:
+<text x="64.77" y="54.61" size="1.016" layer="25" ratio="12" distance="39" rot="R90" align="center-left">NOTE:
 </text>
-<text x="64.77" y="60.6425" size="1.016" layer="25" ratio="12" distance="39" rot="R90" align="center-left">J3-pins must be shorted
-if connector is unused</text>
+<text x="64.77" y="58.7375" size="1.016" layer="25" ratio="12" distance="39" rot="R90" align="center-left">J3-pins must be shorted (or SJ1
+closed) if connector is not used</text>
 <circle x="10" y="80" radius="2.83980625" width="0" layer="41"/>
 <circle x="50" y="60" radius="2.83980625" width="0" layer="41"/>
@@
 <text x="59.3725" y="89.8525" size="0.9652" layer="26" ratio="10" rot="MR90" align="center">+3.3V</text>
 <text x="60.6425" y="91.7575" size="0.9652" layer="26" ratio="10" rot="MR90" align="center">VAPP</text>
+<wire x1="3.8227" y1="39.751" x2="8.8773" y2="39.751" width="0.254" layer="25"/>
+<wire x1="40.6527" y1="39.751" x2="45.7073" y2="39.751" width="0.254" layer="25"/>
 </plain>
 <attributes>
@@
 <attribute name="POPULARITY" value="46" x="-43.18" y="-41.91" size="1.778" layer="27" rot="R270" display="off"/>
 <attribute name="SPICEPREFIX" value="R" x="-43.18" y="-41.91" size="1.778" layer="27" rot="R270" display="off"/>
-<attribute name="VALUE" x="56.7182" y="37.211" size="0.9144" layer="27" ratio="10" rot="R270"/>
+<attribute name="VALUE" x="57.5818" y="33.274" size="0.9144" layer="27" ratio="10" rot="R90"/>
 </element>
 <element name="T1" library="transistor-neu-to92" library_urn="urn:adsk.eagle:library:397" package="TO92" package3d_urn="urn:adsk.eagle:package:28725/2" value="2N2222" x="58.42" y="59.69" smashed="yes">
@@
 <attribute name="MOUSER_PRICE-STOCK" value="https://www.mouser.co.uk/ProductDetail/Harwin/M22-7130542?qs=Jph8NoUxIfVEgwGbmzmPjA%3D%3D" x="62.865" y="83.82" size="1.778" layer="27" rot="R90" display="off"/>
 <attribute name="NAME" x="65.659" y="88.265" size="1.016" layer="25" ratio="10" rot="R90" align="bottom-right"/>
+</element>
+<element name="SJ1" library="jumper" library_urn="urn:adsk.eagle:library:252" package="SJW" package3d_urn="urn:adsk.eagle:package:15507/1" value="No Addon" x="6.35" y="41.275" smashed="yes" rot="MR180">
+<attribute name="NAME" x="9.271" y="42.672" size="1.27" layer="26" ratio="10" rot="MR180"/>
+<attribute name="POPULARITY" value="3" x="6.35" y="41.275" size="1.778" layer="28" rot="MR180" display="off"/>
+<attribute name="VALUE" x="7.35" y="41.275" size="0.02" layer="28" rot="MR180"/>
 </element>
 </elements>
@@
 <wire x1="27.94" y1="38.1" x2="31.115" y2="41.275" width="0.3048" layer="16"/>
 <wire x1="31.115" y1="41.275" x2="42.545" y2="41.275" width="0.3048" layer="16"/>
+<contactref element="SJ1" pad="2"/>
+<wire x1="9.525" y1="39.37" x2="7.62" y2="41.275" width="0.3048" layer="16"/>
+<wire x1="9.525" y1="39.37" x2="9.525" y2="38.1" width="0.3048" layer="16"/>
+<wire x1="9.525" y1="38.1" x2="8.255" y2="36.83" width="0.3048" layer="16"/>
+<wire x1="8.255" y1="36.83" x2="7.62" y2="36.83" width="0.3048" layer="16"/>
 </signal>
 <signal name="MTR-SPEED">
@@
 <wire x1="12.7" y1="66.675" x2="12.7" y2="71.12" width="0.3048" layer="1"/>
 <wire x1="12.7" y1="71.12" x2="20.32" y2="78.74" width="0.3048" layer="1"/>
+<contactref element="SJ1" pad="1"/>
+<wire x1="5.08" y1="41.275" x2="3.175" y2="39.37" width="0.3048" layer="16"/>
+<wire x1="3.175" y1="39.37" x2="3.175" y2="38.1" width="0.3048" layer="16"/>
+<wire x1="4.445" y1="36.83" x2="3.175" y2="38.1" width="0.3048" layer="16"/>
+<wire x1="4.445" y1="36.83" x2="5.08" y2="36.83" width="0.3048" layer="16"/>
 </signal>
 <signal name="SERVO28">
