File: pcb/musicbox/eagle/musicbox.sch (EAGLE design)
At the start: 19 parts, among them J1 1727010, J2 22-27-2031-03, J3 22-27-2021-02, J4 22-27-2021-02, J5 22-27-2051-05, T1 2N2222

Commit message: added gerber files
Parts:
- added SJ1: No Addon, jumper:SJW
Connections:
- net A10: now also SJ1.2
- net N$15: now also SJ1.1
Other:
- moved on the sheet: J3-1
Changed lines of the file:
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@@
 <attribute name="FARNELL_PART_NUMBER" value="1109729"/>
 </part>
+<part name="SJ1" library="jumper" library_urn="urn:adsk.eagle:library:252" deviceset="SJ" device="W" package3d_urn="urn:adsk.eagle:package:15507/1" value="No Addon"/>
 </parts>
 <sheets>
@@
 <attribute name="NAME" x="-55.88" y="57.658" size="1.524" layer="95" rot="MR0"/>
 </instance>
-<instance part="J3" gate="-1" x="86.36" y="152.4" smashed="yes" rot="R270">
-<attribute name="NAME" x="86.36" y="149.098" size="1.524" layer="95"/>
+<instance part="J3" gate="-1" x="91.44" y="152.4" smashed="yes" rot="R270">
+<attribute name="NAME" x="91.44" y="149.098" size="1.524" layer="95"/>
 </instance>
 <instance part="J3" gate="-2" x="81.28" y="152.4" smashed="yes" rot="R270">
@@
 <attribute name="VALUE" x="6.35" y="129.54" size="1.778" layer="96" rot="R180"/>
 <attribute name="NAME" x="6.35" y="105.918" size="1.778" layer="95" rot="R180"/>
+</instance>
+<instance part="SJ1" gate="1" x="86.36" y="160.02" smashed="yes">
+<attribute name="NAME" x="83.82" y="162.56" size="1.778" layer="95"/>
+<attribute name="VALUE" x="83.82" y="156.21" size="1.778" layer="96"/>
 </instance>
 </instances>
@@
 </segment>
 <segment>
-<wire x1="86.36" y1="154.94" x2="91.44" y2="154.94" width="0.1524" layer="91"/>
-<label x="91.44" y="154.94" size="1.4224" layer="95" xref="yes"/>
+<wire x1="91.44" y1="154.94" x2="93.98" y2="154.94" width="0.1524" layer="91"/>
+<label x="96.52" y="154.94" size="1.4224" layer="95" xref="yes"/>
 <pinref part="J3" gate="-1" pin="S"/>
+<pinref part="SJ1" gate="1" pin="2"/>
+<wire x1="93.98" y1="154.94" x2="96.52" y2="154.94" width="0.1524" layer="91"/>
+<wire x1="91.44" y1="160.02" x2="93.98" y2="160.02" width="0.1524" layer="91"/>
+<wire x1="93.98" y1="160.02" x2="93.98" y2="154.94" width="0.1524" layer="91"/>
+<junction x="93.98" y="154.94"/>
 </segment>
 </net>
@@
 <pinref part="U$1" gate="G$1" pin="PA10"/>
 <pinref part="J3" gate="-2" pin="S"/>
-<wire x1="81.28" y1="154.94" x2="53.34" y2="154.94" width="0.1524" layer="91"/>
-</segment>
-</net>
+<wire x1="81.28" y1="154.94" x2="78.74" y2="154.94" width="0.1524" layer="91"/>
+<pinref part="SJ1" gate="1" pin="1"/>
+<wire x1="78.74" y1="154.94" x2="53.34" y2="154.94" width="0.1524" layer="91"/>
+<wire x1="81.28" y1="160.02" x2="78.74" y2="160.02" width="0.1524" layer="91"/>
+<wire x1="78.74" y1="160.02" x2="78.74" y2="154.94" width="0.1524" layer="91"/>
+<junction x="78.74" y="154.94"/>
+</segment>
+</net>
